File: ads1299_test_board/ads1299.kicad_sch (KiCad schematic)
At the start: 20 parts, among them U1 ADS1299

Commit message: power circuit
Connections:
- net GNDA renamed agnd
- net GNDD renamed dgnd
Changed lines of the file:
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@@
 		(polyline
 			(pts
-				(xy 19.05 89.8524) (xy 45.72 90.17) (xy 45.72 158.75) (xy 42.545 162.56) (xy 20.955 162.56) (xy 19.05 158.75)
+				(xy 19.05 89.8524) (xy 45.72 90.17) (xy 45.72 158.75) (xy 42.545 161.29) (xy 20.955 161.29) (xy 19.05 158.75)
 			)
 			(stroke
@@
 		(in_pos_files yes)
 		(dnp no)
-		(fields_autoplaced yes)
 		(property "Reference" "#PWR04"
 			(at 99.06 143.51 0)
@@
 			)
 		)
-		(property "Value" "GNDD"
-			(at 99.06 140.97 0)
-			(show_name no)
-			(do_not_autoplace no)
-			(effects
-				(font
-					(size 1.27 1.27)
-				)
+		(property "Value" "dgnd"
+			(at 97.028 141.224 0)
+			(show_name no)
+			(do_not_autoplace no)
+			(effects
+				(font
+					(size 1.27 1.27)
+				)
+				(justify left)
 			)
 		)
@@
 		(in_pos_files yes)
 		(dnp no)
-		(fields_autoplaced yes)
 		(property "Reference" "#PWR08"
 			(at 25.4 130.81 0)
@@
 			)
 		)
-		(property "Value" "GNDA"
-			(at 25.4 129.54 0)
-			(show_name no)
-			(do_not_autoplace no)
-			(effects
-				(font
-					(size 1.27 1.27)
-				)
+		(property "Value" "agnd"
+			(at 25.146 129.286 0)
+			(show_name no)
+			(do_not_autoplace no)
+			(effects
+				(font
+					(size 1.27 1.27)
+				)
+				(justify left)
 			)
 		)
@@
 			)
 		)
-		(property "Value" "GNDA"
-			(at 25.4 109.22 0)
-			(show_name no)
-			(do_not_autoplace no)
-			(effects
-				(font
-					(size 1.27 1.27)
-				)
+		(property "Value" "agnd"
+			(at 27.94 105.4099 0)
+			(show_name no)
+			(do_not_autoplace no)
+			(effects
+				(font
+					(size 1.27 1.27)
+				)
+				(justify left)
 			)
 		)
@@
 		(in_pos_files yes)
 		(dnp no)
-		(fields_autoplaced yes)
 		(property "Reference" "#PWR09"
 			(at 25.4 140.97 0)
@@
 			)
 		)
-		(property "Value" "GNDA"
-			(at 25.4 139.7 0)
-			(show_name no)
-			(do_not_autoplace no)
-			(effects
-				(font
-					(size 1.27 1.27)
-				)
+		(property "Value" "agnd"
+			(at 25.146 139.446 0)
+			(show_name no)
+			(do_not_autoplace no)
+			(effects
+				(font
+					(size 1.27 1.27)
+				)
+				(justify left)
 			)
 		)
@@
 			)
 		)
-		(property "Value" "GNDA"
-			(at 26.67 157.48 0)
-			(show_name no)
-			(do_not_autoplace no)
-			(effects
-				(font
-					(size 1.27 1.27)
-				)
+		(property "Value" "agnd"
+			(at 29.21 153.6699 0)
+			(show_name no)
+			(do_not_autoplace no)
+			(effects
+				(font
+					(size 1.27 1.27)
+				)
+				(justify left)
 			)
 		)
@@
 		(in_pos_files yes)
 		(dnp no)
-		(fields_autoplaced yes)
 		(property "Reference" "#PWR05"
 			(at 26.67 101.6 0)
@@
 			)
 		)
-		(property "Value" "GNDA"
-			(at 26.67 100.33 0)
-			(show_name no)
-			(do_not_autoplace no)
-			(effects
-				(font
-					(size 1.27 1.27)
-				)
+		(property "Value" "agnd"
+			(at 24.892 100.076 0)
+			(show_name no)
+			(do_not_autoplace no)
+			(effects
+				(font
+					(size 1.27 1.27)
+				)
+				(justify left)
 			)
 		)
@@
 		(in_pos_files yes)
 		(dnp no)
-		(fields_autoplaced yes)
 		(property "Reference" "#PWR03"
 			(at 93.98 143.51 0)
@@
 			)
 		)
-		(property "Value" "GNDA"
-			(at 93.98 142.24 0)
-			(show_name no)
-			(do_not_autoplace no)
-			(effects
-				(font
-					(size 1.27 1.27)
-				)
-			)
-		)
+		(property "Value" "agnd"
+			(at 90.932 141.224 0)
+			(show_name no)
+			(do_not_autoplace no)
+			(effects
+				(font
+					(size 1.27 1.27)
+				)
+				(justify left)
+			)
+		)
