File: ads1299_test_board/ads1299.kicad_sch (KiCad schematic)
At the start: 29 parts, among them U1 ADS1299, U4 OPA376xxD

Commit message: PCB design charger and power supply
Parts:
- added R27, R28, R29, R30: 10k, Resistor_SMD:R_0402_1005Metric_Pad0.72x0.64mm_HandSolder, symbol Device:R
Connections:
- net GND: now also R27.1, R28.1, R29.1, R30.1
- net GPIO1: no longer names the net of U1.42 (GPIO1)
- net GPIO1: now also R27.2
- net GPIO2: no longer names the net of U1.44 (GPIO2)
- net GPIO2: now also R28.2
- net GPIO3: no longer names the net of U1.45 (GPIO3)
- net GPIO3: now also R29.2
- net GPIO4: no longer names the net of U1.46 (GPIO4)
- net GPIO4: now also R30.2

Commit message: pcb design
Parts:
- removed C2, C3, C4, C5: 0.15uF, Capacitor_SMD:C_0603_1608Metric_Pad1.08x0.95mm_HandSolder, symbol Device:C_US
- removed R1, R2, R3, R4, R5, R6, R7, R8: 10K, Resistor_SMD:R_0402_1005Metric_Pad0.72x0.64mm_HandSolder, symbol Device:R_US
- added CN1, CN2: W2A45C103MAT2A, W2A45C103MAT2A:W2A45C103MAT2A, symbol W2A45C103MAT2A:W2A45C103MAT2A
- added J3: Conn_02x05_Top_Bottom, Connector_Molex:Molex_Mini-Fit_Jr_5566-10A_2x05_P4.20mm_Vertical, symbol Connector_Generic:Conn_02x05_Top_Bottom
- added R23, R31: CAY16-2201F4LF, CAY16-2201F4LF:RESCAX80P160X320X60-8N, symbol CAY16-2201F4LF:CAY16-2201F4LF
Connections:
- net 1N: now also CN1.7, R31.2
- net 1P: now also CN1.8, R31.1
- net 2N: now also CN1.5, R31.4
- net 2P: now also CN1.6, R31.3
- net 3N: now also CN2.7, R23.2
- net 3P: now also CN2.8, R23.1
- net 4N: now also CN2.5, R23.4
- net 4P: now also CN2.6, R23.3
- net Bias_electrode: now also J3.10 (Pin_10)
- net GND: now also CN1.1, CN1.2, CN1.3, CN1.4, CN2.1, CN2.2, CN2.3, CN2.4; no longer U1.18 (SRB2)
- net Ref_electrode: now also J3.5 (Pin_5)
- new net IN1N: J3.1 (Pin_1), R31.7
- new net IN1P: J3.6 (Pin_6), R31.8
- new net IN2N: J3.2 (Pin_2), R31.5
- new net IN2P: J3.7 (Pin_7), R31.6
- new net IN3N: J3.3 (Pin_3), R23.7
- new net IN3P: J3.8 (Pin_8), R23.8
- new net IN4N: J3.4 (Pin_4), R23.5
- new net IN4P: J3.9 (Pin_9), R23.6
- no-connect marks 0 -> 1
Other:
- moved on the sheet: R22
