File: ads1299_test_board/ads1299.kicad_sch (KiCad schematic)
At the start: 26 parts, among them CN1 W2A45C103MAT2A, CN2 W2A45C103MAT2A, J3 Conn_02x05_Top_Bottom, U1 ADS1299, U4 OPA376xxD

Commit message: work on PCB
Connections:
- net Bias_electrode: now also J3.1 (Pin_1); no longer J3.10 (Pin_10)
- net IN1N: now also J3.2 (Pin_2); no longer J3.1 (Pin_1)
- net IN1P: now also J3.7 (Pin_7); no longer J3.6 (Pin_6)
- net IN2N: now also J3.3 (Pin_3); no longer J3.2 (Pin_2)
- net IN2P: now also J3.8 (Pin_8); no longer J3.7 (Pin_7)
- net IN3N: now also J3.4 (Pin_4); no longer J3.3 (Pin_3)
- net IN3P: now also J3.9 (Pin_9); no longer J3.8 (Pin_8)
- net IN4N: now also J3.5 (Pin_5); no longer J3.4 (Pin_4)
- net IN4P: now also J3.10 (Pin_10); no longer J3.9 (Pin_9)
- net Ref_electrode: now also J3.6 (Pin_6); no longer J3.5 (Pin_5)
- no-connect marks 1 -> 3
Changed lines of the file:
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@@
 	)
 	(no_connect
+		(at 151.13 118.11)
+	)
+	(no_connect
+		(at 151.13 115.57)
+	)
+	(no_connect
 		(at 151.13 62.23)
 	)
@@
 	(wire
 		(pts
-			(xy 31.75 100.33) (xy 34.29 100.33)
-		)
-		(stroke
-			(width 0)
-			(type default)
-		)
-	)
-	(wire
-		(pts
 			(xy 151.13 87.63) (xy 153.67 87.63)
 		)
@@
 	)
 	(label "IN1N"
-		(at 44.45 90.17 0)
+		(at 44.45 92.71 0)
 		(effects
 			(font
@@
 	)
 	(label "IN3P"
-		(at 31.75 95.25 180)
+		(at 31.75 97.79 180)
 		(effects
 			(font
@@
 	)
 	(label "Bias_electrode"
-		(at 34.29 100.33 180)
+		(at 44.45 90.17 0)
 		(effects
 			(font
 				(size 1.27 1.27)
 			)
-			(justify right bottom)
+			(justify left bottom)
 		)
 	)
@@
 	)
 	(label "IN4P"
-		(at 31.75 97.79 180)
+		(at 31.75 100.33 180)
 		(effects
 			(font
@@
 	)
 	(label "Ref_electrode"
-		(at 44.45 100.33 0)
+		(at 31.75 90.17 180)
 		(effects
 			(font
 				(size 1.27 1.27)
 			)
-			(justify left bottom)
+			(justify right bottom)
 		)
 	)
@@
 	)
 	(label "IN4N"
-		(at 44.45 97.79 0)
+		(at 44.45 100.33 0)
 		(effects
 			(font
@@
 	)
 	(label "IN3N"
-		(at 44.45 95.25 0)
+		(at 44.45 97.79 0)
 		(effects
 			(font
@@
 	)
 	(label "IN1P"
-		(at 31.75 90.17 180)
+		(at 31.75 92.71 180)
 		(effects
 			(font
@@
 	)
 	(label "IN2P"
-		(at 31.75 92.71 180)
+		(at 31.75 95.25 180)
 		(effects
 			(font
@@
 	)
 	(label "IN2N"
-		(at 44.45 92.71 0)
+		(at 44.45 95.25 0)
 		(effects
 			(font
@@
 			"b6c532a8-276a-4ea5-9017-38b21cdc40b9" "bce87beb-76ab-415f-add4-ecb5c5e76c9d"
 			"c1d2e623-7db4-4274-b8ce-083743e258fa" "c503ab81-7469-4442-9a38-691380bce035"
-			"c99cc4d9-7dd4-45c9-899b-2092c104cade" "cc340a1a-22e8-4165-bca6-8721b8b0b063"
-			"cdb295c9-1868-48e4-a0c6-508198fb6fdd" "d1b63223-74ee-4fce-b3ad-c32cb9f1cd8e"
-			"d587d880-0af7-4162-aed2-ce590c43f627" "d80cd447-9bd6-4eeb-a66f-8bda6f73d70c"
-			"d82f30f3-4065-43b6-81c8-9b403b9c8be6" "e6ed5087-4183-43e8-b7d2-9a02f45edc66"
-			"eea9b404-53bd-45ab-b143-c46d4d461be0" "f128c97a-0b12-446a-9f99-d13d1a6daf4d"
-			"f17a7fb9-c9c7-4438-b337-270b728fc4eb" "f4253d6f-c0a3-40e9-9ad7-db83303dc0c0"
-			"f4e87d51-f4f5-4b36-b6f0-fb2239fd7979" "fa5b47de-801c-4761-919e-876be397dbb4"
-			"fb528be8-a716-4c16-8d97-8b87115554fd"
+			"cc340a1a-22e8-4165-bca6-8721b8b0b063" "cdb295c9-1868-48e4-a0c6-508198fb6fdd"
+			"d1b63223-74ee-4fce-b3ad-c32cb9f1cd8e" "d587d880-0af7-4162-aed2-ce590c43f627"
+			"d80cd447-9bd6-4eeb-a66f-8bda6f73d70c" "d82f30f3-4065-43b6-81c8-9b403b9c8be6"
+			"e6ed5087-4183-43e8-b7d2-9a02f45edc66" "eea9b404-53bd-45ab-b143-c46d4d461be0"
+			"f128c97a-0b12-446a-9f99-d13d1a6daf4d" "f17a7fb9-c9c7-4438-b337-270b728fc4eb"
+			"f4253d6f-c0a3-40e9-9ad7-db83303dc0c0" "f4e87d51-f4f5-4b36-b6f0-fb2239fd7979"
+			"fa5b47de-801c-4761-919e-876be397dbb4" "fb528be8-a716-4c16-8d97-8b87115554fd"
 		)
 	)

Commit message: final form
Parts:
- removed R19: 10k, Resistor_SMD:R_0402_1005Metric_Pad0.72x0.64mm_HandSolder, symbol Device:R_Variable
- added R19: 10k, Resistor_SMD:R_0402_1005Metric_Pad0.72x0.64mm_HandSolder, symbol Device:R
- C26: value C -> 15nF; footprint (none) -> Capacitor_SMD:C_0402_1005Metric_Pad0.74x0.62mm_HandSolder
- R25: value R -> 1M; footprint (none) -> Resistor_SMD:R_0402_1005Metric_Pad0.72x0.64mm_HandSolder
- TP1: footprint TestPoint:TestPoint_Pad_D1.5mm -> TestPoint:TestPoint_Pad_D1.0mm
Connections:
- net GND: now also R19.2
- net at R12.2, U1.60 (BIASREF): now also R19.1
Changed lines of the file:
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@@
 	)
 	(symbol
-		(lib_id "Device:R_Variable")
+		(lib_id "Device:R")
 		(at 187.96 63.5 0)
 		(unit 1)
@@
 		(fields_autoplaced yes)
 		(property "Reference" "R19"
-			(at 191.77 62.2299 0)
+			(at 190.5 62.2299 0)
 			(show_name no)
 			(do_not_autoplace no)
@@
 		)
 		(property "Value" "10k"
-			(at 191.77 64.7699 0)
+			(at 190.5 64.7699 0)
 			(show_name no)
 			(do_not_autoplace no)
@@
 			)
 		)
-		(property "Description" "Variable resistor"
+		(property "Description" "Resistor"
 			(at 187.96 63.5 0)
 			(hide yes)
@@
 			)
 		)
+		(pin "1"
+		)
 		(pin "2"
-		)
-		(pin "1"
 		)
 		(instances
@@
 			)
 		)
-		(property "Footprint" "TestPoint:TestPoint_Pad_D1.5mm"
+		(property "Footprint" "TestPoint:TestPoint_Pad_D1.0mm"
 			(at 167.64 101.6 0)
 			(hide yes)
@@
 			)
 		)
-		(property "Value" "C"
+		(property "Value" "15nF"
 			(at 163.83 39.37 90)
 			(show_name no)
@@
 			)
 		)
-		(property "Footprint" ""
+		(property "Footprint" "Capacitor_SMD:C_0402_1005Metric_Pad0.74x0.62mm_HandSolder"
 			(at 167.64 43.4848 0)
 			(hide yes)
@@
 			)
 		)
-		(property "Value" "R"
+		(property "Value" "1M"
 			(at 173.228 51.054 90)
 			(show_name no)
@@
 			)
 		)
-		(property "Footprint" ""
+		(property "Footprint" "Resistor_SMD:R_0402_1005Metric_Pad0.72x0.64mm_HandSolder"
 			(at 163.83 47.752 90)
 			(hide yes)

Commit message: 8 channel
Parts:
- removed J3: Conn_02x05_Top_Bottom, Connector_Molex:Molex_Mini-Fit_Jr_5566-10A_2x05_P4.20mm_Vertical, symbol Connector_Generic:Conn_02x05_Top_Bottom
- added CN3, CN4: W2A45C103MAT2A, W2A45C103MAT2A:W2A45C103MAT2A, symbol W2A45C103MAT2A:W2A45C103MAT2A
- added J2: Conn_02x10_Counter_Clockwise, Connector_IDC:IDC-Header_2x10_P2.54mm_Vertical, symbol Connector_Generic:Conn_02x10_Counter_Clockwise
- added R32, R33: CAY16-2201F4LF, CAY16-2201F4LF:RESCAX80P160X320X60-8N, symbol CAY16-2201F4LF:CAY16-2201F4LF
Connections:
- net +5V: now also J2.19 (Pin_19), J2.20 (Pin_20); no longer U1.1 (IN8N), U1.2 (IN8P), U1.3 (IN7N), U1.4 (IN7P), U1.5 (IN6N), U1.6 (IN6P), U1.7 (IN5N), U1.8 (IN5P)
- net 1N: now also CN1.6; no longer CN1.7
- net 1P: now also CN1.5; no longer CN1.8
- net 2N: now also CN1.8; no longer CN1.5
- net 2P: now also CN1.7; no longer CN1.6
- net 3N: now also CN2.6; no longer CN2.7
- net 3P: now also CN2.5; no longer CN2.8
- net 4N: now also CN2.8; no longer CN2.5
- net 4P: now also CN2.7; no longer CN2.6
- net Bias_electrode: now also J2.18 (Pin_18)
- net GND: now also CN3.1, CN3.2, CN3.3, CN3.4, CN4.1, CN4.2, CN4.3, CN4.4
- net IN1N: now also J2.2 (Pin_2)
- net IN1P: now also J2.1 (Pin_1)
- net IN2N: now also J2.4 (Pin_4)
- net IN2P: now also J2.3 (Pin_3)
- net IN3N: now also J2.6 (Pin_6)
- net IN3P: now also J2.5 (Pin_5)
- net IN4N: now also J2.8 (Pin_8)
- net IN4P: now also J2.7 (Pin_7)
- net Ref_electrode: now also J2.17 (Pin_17)
- new net 5N: CN3.6, R33.2, U1.7 (IN5N)
- new net 5P: CN3.5, R33.1, U1.8 (IN5P)
- new net 6N: CN3.8, R33.4, U1.5 (IN6N)
- new net 6P: CN3.7, R33.3, U1.6 (IN6P)
- new net 7N: CN4.6, R32.2, U1.3 (IN7N)
- new net 7P: CN4.5, R32.1, U1.4 (IN7P)
- new net 8N: CN4.8, R32.4, U1.1 (IN8N)
- new net 8P: CN4.7, R32.3, U1.2 (IN8P)
- new net IN5N: J2.10 (Pin_10), R33.7
- new net IN5P: J2.9 (Pin_9), R33.8
- new net IN6N: J2.12 (Pin_12), R33.5
- new net IN6P: J2.11 (Pin_11), R33.6
- new net IN7N: J2.14 (Pin_14), R32.7
- new net IN7P: J2.13 (Pin_13), R32.8
- new net IN8N: J2.16 (Pin_16), R32.5
- new net IN8P: J2.15 (Pin_15), R32.6
Other:
- moved on the sheet: CN1, CN2, R23, R31

Commit message: op-amp sot23-5
Parts:
- removed U4: OPA376xxD, Package_SO:SOIC-8_3.9x4.9mm_P1.27mm, symbol Amplifier_Operational:OPA376xxD
- added U5: OPA376xxDBV, Package_TO_SOT_SMD:SOT-23-5, symbol Amplifier_Operational:OPA376xxDBV
Connections:
- net +5V: now also U5.5 (V+)
- net GND: now also U5.2 (V-)
- net Ref_electrode: now also U5.3 (+)
- net SRB1: now also U5.1, U5.4 (-)
Changed lines of the file:
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@@
-	)
-	(symbol
-		(lib_id "Amplifier_Operational:OPA376xxD")
-		(at 78.74 177.8 0)
-		(unit 1)
-		(body_style 1)
-		(exclude_from_sim no)
-		(in_bom yes)
-		(on_board yes)
-		(in_pos_files yes)
-		(dnp no)
-		(fields_autoplaced yes)
-		(property "Reference" "U4"
-			(at 73.0819 187.96 0)
-			(show_name no)
-			(do_not_autoplace no)
-			(effects
-				(font
-					(size 1.27 1.27)
-				)
-				(justify right)
-			)
-		)
-		(property "Value" "OPA376xxD"
-			(at 73.0819 185.42 0)
-			(show_name no)
-			(do_not_autoplace no)
-			(effects
-				(font
-					(size 1.27 1.27)
-				)
-				(justify right)
-			)
-		)
-		(property "Footprint" "Package_SO:SOIC-8_3.9x4.9mm_P1.27mm"
-			(at 76.2 182.88 0)
-			(hide yes)
-			(show_name no)
-			(do_not_autoplace no)
-			(effects
-				(font
-					(size 1.27 1.27)
-				)
-				(justify left)
-			)
-		)
-		(property "Datasheet" "http://www.ti.com/lit/ds/symlink/opa376.pdf"
-			(at 82.55 173.99 0)
-			(hide yes)
-			(show_name no)
-			(do_not_autoplace no)
-			(effects
-				(font
-					(size 1.27 1.27)
-				)
-			)
-		)
-		(property "Description" "Single Low-Noise, Low Quiescent Current, Precision Operational Amplifier e-trim Series, SOIC-8"
-			(at 78.74 177.8 0)
-			(hide yes)
-			(show_name no)
-			(do_not_autoplace no)
-			(effects
-				(font
-					(size 1.27 1.27)
-				)
-			)
-		)
-		(pin "4"
-		)
-		(pin "6"
-		)
-		(pin "5"
-		)
-		(pin "1"
-		)
-		(pin "2"
-		)
-		(pin "7"
-		)
-		(pin "3"
-		)
-		(pin "8"
-		)
-		(instances
-			(project "ads1299_test_board"
-				(path "/97f9a33a-d3bd-406a-9672-b92babffe6b5/fc0c8262-5909-4fc3-abb1-3b11f752dbb7"
-					(reference "U4")
-					(unit 1)
-				)
-			)
-		)
 	)
 	(symbol
@@
 				(path "/97f9a33a-d3bd-406a-9672-b92babffe6b5/fc0c8262-5909-4fc3-abb1-3b11f752dbb7"
 					(reference "R22")
+					(unit 1)
+				)
+			)
+		)
+	)
+	(symbol
+		(lib_id "Amplifier_Operational:OPA376xxDBV")
+		(at 78.74 177.8 0)
+		(unit 1)
+		(body_style 1)
+		(exclude_from_sim no)
+		(in_bom yes)
+		(on_board yes)
+		(in_pos_files yes)
+		(dnp no)
+		(fields_autoplaced yes)
+		(property "Reference" "U5"
+			(at 91.44 171.3798 0)
+			(show_name no)
+			(do_not_autoplace no)
+			(effects
+				(font
+					(size 1.27 1.27)
+				)
+			)
+		)
+		(property "Value" "OPA376xxDBV"
+			(at 91.44 173.9198 0)
+			(show_name no)
+			(do_not_autoplace no)
+			(effects
+				(font
+					(size 1.27 1.27)
+				)
+			)
+		)
+		(property "Footprint" "Package_TO_SOT_SMD:SOT-23-5"
+			(at 76.2 182.88 0)
+			(hide yes)
+			(show_name no)
+			(do_not_autoplace no)
+			(effects
+				(font
+					(size 1.27 1.27)
+				)
+				(justify left)
+			)
+		)
+		(property "Datasheet" "http://www.ti.com/lit/ds/symlink/opa376.pdf"
+			(at 78.74 172.72 0)
+			(hide yes)
+			(show_name no)
+			(do_not_autoplace no)
+			(effects
+				(font
+					(size 1.27 1.27)
+				)
+			)
+		)
+		(property "Description" "Single Low-Noise, Low Quiescent Current, Precision Operational Amplifier e-trim Series, SOT-23-5"
+			(at 78.74 177.8 0)
+			(hide yes)
+			(show_name no)
+			(do_not_autoplace no)
+			(effects
+				(font
+					(size 1.27 1.27)
+				)
+			)
+		)
+		(pin "4"
+		)
+		(pin "3"
+		)
+		(pin "1"
+		)
+		(pin "2"
+		)
+		(pin "5"
+		)
+		(instances
+			(project "ads1299_test_board"
+				(path "/97f9a33a-d3bd-406a-9672-b92babffe6b5/fc0c8262-5909-4fc3-abb1-3b11f752dbb7"
+					(reference "U5")
 					(unit 1)
 				)
@@
 		)
 	)
-	(group ""
-		(members "046aa602-50ba-496a-820d-bffa0f107be9" "13f3651d-cba0-47a1-9456-a9714d8f9410"
-			"167a5735-2a7b-4998-bf8c-63d231675a37" "1b2f03a5-2bd0-449f-ac2d-7d29bde24763"
-			"3c6cbad6-83ac-4331-b944-242164102515" "42a4158f-b89c-4126-93dc-0c2f290adbe9"
-			"53af7c84-ebeb-407d-9427-de8471a3e76d" "5581943d-d43c-401b-8314-2912403fe7a4"
-			"57d983db-a91f-4db6-aeee-e696adca4886" "63825c48-cbd1-489d-954a-37ce0e07d92f"
-			"67fc5cc0-d23a-438c-a1b1-9d78c1aa4743" "8ef13d0f-13c7-4f0b-95dc-83441b281058"
-			"ade85c43-0cb2-4d35-a5c1-ce17b09ed102" "c60f8070-fed3-49d7-b743-96fce6d7d286"
-			"cfbe0bc2-6aad-4f8e-82cc-7ee471172378" "d21aed29-08cc-4a30-af28-817b09461db7"
-			"d89643ed-de0e-41d4-bcaf-f1965adcd533" "d8db8a3f-be9d-4663-9470-e93812c8abbc"
-			"e7794fe5-da48-480e-97fb-42bdc85875e2" "e86411de-ecff-4a34-b715-fde9c47f3fc9"
-			"f1d32478-0ca0-4ae3-af94-201fe5968825" "f76b8b52-a39b-480a-8af0-95fb8945d6bb"
-		)
-	)
