File: ads1299_test_board/charger.kicad_sch (KiCad schematic)
At the start: 8 parts, among them Q1 AO3407A, U2 MCP73832-2-OT

Commit message: power circuit
Connections:
- net bat_gnd renamed agnd
Changed lines of the file:
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@@
 			)
 		)
-		(property "Value" "bat_gnd"
+		(property "Value" "agnd"
 			(at 138.43 60.198 0)
 			(show_name no)
@@
 			)
 		)
-		(property "Value" "bat_gnd"
-			(at 100.33 80.01 0)
-			(show_name no)
-			(do_not_autoplace no)
-			(effects
-				(font
-					(size 1.27 1.27)
-				)
+		(property "Value" "agnd"
+			(at 102.87 76.1999 0)
+			(show_name no)
+			(do_not_autoplace no)
+			(effects
+				(font
+					(size 1.27 1.27)
+				)
+				(justify left)
 			)
 		)
@@
 			)
 		)
-		(property "Value" "bat_gnd"
+		(property "Value" "agnd"
 			(at 86.36 68.58 0)
 			(show_name no)
@@
 			)
 		)
-		(property "Value" "bat_gnd"
-			(at 95.25 68.58 0)
-			(show_name no)
-			(do_not_autoplace no)
-			(effects
-				(font
-					(size 1.27 1.27)
-				)
-			)
-		)
+		(property "Value" "agnd"
+			(at 97.79 64.7699 0)
+			(show_name no)
+			(do_not_autoplace no)
+			(effects
+				(font
+					(size 1.27 1.27)
+				)
+				(justify left)
+			)
+		)
