File: ads1299_test_board/charger.kicad_sch (KiCad schematic)
At the start: 11 parts, among them J1 Conn_01x02, Q1 AO3407A, U2 MCP73832-2-OT

Commit message: PCB design charger and power supply
Connections:
- net Vusb_charge is gone; now on net Vusb: C12.1, D1.2 (A), D2.2 (A), R11.2, U2.4 (V_{DD})
- net Vusb: no longer D2.1 (K), Q1.1 (G)
- new net: D2.1 (K), Q1.1 (G)
Changed lines of the file:
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@@
 	(paper "A4")
 	(junction
-		(at 125.73 88.9)
-		(diameter 0)
-		(color 0 0 0 0)
-	)
-	(junction
 		(at 167.64 77.47)
 		(diameter 0)
@@
 	(wire
 		(pts
-			(xy 125.73 88.9) (xy 125.73 101.6)
-		)
-		(stroke
-			(width 0)
-			(type default)
-		)
-	)
-	(wire
-		(pts
 			(xy 137.16 88.9) (xy 142.24 88.9)
 		)
@@
 	(wire
 		(pts
-			(xy 119.38 88.9) (xy 125.73 88.9)
+			(xy 119.38 88.9) (xy 129.54 88.9)
 		)
 		(stroke
@@
 	(wire
 		(pts
-			(xy 125.73 88.9) (xy 129.54 88.9)
-		)
-		(stroke
-			(width 0)
-			(type default)
-		)
-	)
-	(wire
-		(pts
 			(xy 111.76 80.01) (xy 111.76 83.82)
 		)
@@
 			(width 0)
 			(type default)
-		)
-	)
-	(wire
-		(pts
-			(xy 110.49 101.6) (xy 125.73 101.6)
-		)
-		(stroke
-			(width 0)
-			(type default)
-		)
-	)
-	(hierarchical_label "Vusb"
-		(shape input)
-		(at 110.49 101.6 180)
-		(effects
-			(font
-				(size 1.27 1.27)
-			)
-			(justify right)
 		)
 	)
@@
 		)
 	)
-	(hierarchical_label "Vusb_charge"
+	(hierarchical_label "Vusb"
 		(shape input)
 		(at 166.37 77.47 180)
