File: ads1299_test_board/power_circuit.kicad_sch (KiCad schematic)
At the start: 7 parts, among them U3 TPS61023DRLR, U4 AP2112K-3.3, U5 TPS7A20xxxDBV

Commit message: Added spiro's schematic to project. Also added lib folder
Parts:
- removed C14: C, symbol Device:C
- removed L1: L, symbol Device:L
- removed R12: R, symbol Device:R
- removed U3: TPS61023DRLR, TPS61023DRLR:SOT563-ORI, symbol TPS61023DRLR:TPS61023DRLR
- removed U4: AP2112K-3.3, Package_TO_SOT_SMD:SOT-23-5, symbol Regulator_Linear:AP2112K-3.3
- removed U5: TPS7A20xxxDBV, Package_TO_SOT_SMD:SOT-23-5, symbol Regulator_Linear:TPS7A20xxxDBV
- added C15: 200p, symbol Device:C
- added C16: 10u, symbol Device:C
- added C17, C18, C19: 20u, symbol Device:C
- added F1: Fuse, symbol Device:Fuse
- added IC1: TPS61023DRLR, SOTFL50P160X60-6N, symbol TPS61023DRLR:TPS61023DRLR
- added IC2: TPS7A2030PDBVR, SOT95P280X145-5N, symbol TPS7A2030PDBVR:TPS7A2030PDBVR
- added J1: Conn_01x02, symbol Connector_Generic:Conn_01x02
- added L2: 2.2u, symbol Device:L
- added R14: 100k, symbol Device:R
- added R15, R17, R18: R, symbol Device:R
- added R16: 825k, symbol Device:R
- added SW1: SW_Push, symbol Switch:SW_Push
- added U6: AP2112K-3.3, Package_TO_SOT_SMD:SOT-23-5, symbol Regulator_Linear:AP2112K-3.3
Connections:
- new net: IC1.2 (EN), R15.2
- new net: C16.1, IC1.4 (GND), L2.1
- new net: C15.2, R14.1, R16.2
- new net: R18.1, U6.3 (EN)
- new net: R15.1, SW1.1
- new net: F1.2, J1.2 (Pin_2)
- new net +3.3V: U6.5 (VOUT)
- new net +BATT: F1.1, SW1.2
- new net -BATT: C16.2, C17.2, C18.2, C19.2, J1.1 (Pin_1), R14.2, U6.2 (GND)
- new net SW: IC1.6 (VOUT), L2.2
- new net VCC: C15.1, C17.1, C18.1, C19.1, R16.1, R17.2, R18.2, U6.1 (VIN)
Other:
- moved on the sheet: R13
