File: ads1299_test_board/power_circuit.kicad_sch (KiCad schematic)
At the start: 16 parts, among them IC1 TPS61023DRLR, IC2 TPS7A2050PDBVR, SW1 EG1218, U6 AP2112K-3.3

Commit message: final form
Parts:
- removed R13: 0, symbol Device:R
Changed lines of the file:
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@@
-	)
-	(symbol
-		(lib_id "Device:R")
-		(at 83.82 124.46 90)
-		(unit 1)
-		(body_style 1)
-		(exclude_from_sim no)
-		(in_bom yes)
-		(on_board yes)
-		(in_pos_files yes)
-		(dnp no)
-		(fields_autoplaced yes)
-		(property "Reference" "R13"
-			(at 83.82 118.11 90)
-			(show_name no)
-			(do_not_autoplace no)
-			(effects
-				(font
-					(size 1.27 1.27)
-				)
-			)
-		)
-		(property "Value" "0"
-			(at 83.82 120.65 90)
-			(show_name no)
-			(do_not_autoplace no)
-			(effects
-				(font
-					(size 1.27 1.27)
-				)
-			)
-		)
-		(property "Footprint" ""
-			(at 83.82 126.238 90)
-			(hide yes)
-			(show_name no)
-			(do_not_autoplace no)
-			(effects
-				(font
-					(size 1.27 1.27)
-				)
-			)
-		)
-		(property "Datasheet" ""
-			(at 83.82 124.46 0)
-			(hide yes)
-			(show_name no)
-			(do_not_autoplace no)
-			(effects
-				(font
-					(size 1.27 1.27)
-				)
-			)
-		)
-		(property "Description" "Resistor"
-			(at 83.82 124.46 0)
-			(hide yes)
-			(show_name no)
-			(do_not_autoplace no)
-			(effects
-				(font
-					(size 1.27 1.27)
-				)
-			)
-		)
-		(pin "2"
-		)
-		(pin "1"
-		)
-		(instances
-			(project "ads1299_test_board"
-				(path "/97f9a33a-d3bd-406a-9672-b92babffe6b5/a537b4c0-2d82-4fbb-91d8-e3a7ef64a59b"
-					(reference "R13")
-					(unit 1)
-				)
-			)
-		)
 	)
 	(symbol

Commit message: fuse and 1ohm r
Parts:
- added F1: Fuse_Small, Fuse:Fuse_2512_6332Metric_Pad1.52x3.35mm_HandSolder, symbol Device:Fuse_Small
Connections:
- net GNDD is gone; now on net GND: U6.2 (GND)
- net VCC: now also F1.1; no longer C15.1, C17.1, C18.1, C19.1, IC1.6 (VOUT), R16.1
- net at R15.1: now also SW1.2 (C); no longer SW1.3 (A)
- new net: C15.1, C17.1, C18.1, C19.1, F1.2, IC1.6 (VOUT), R16.1
Other:
- moved on the sheet: SW1
Changed lines of the file:
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@@
+	)
+	(junction
+		(at 167.64 85.09)
+		(diameter 0)
+		(color 0 0 0 0)
 	)
 	(junction
@@
 	)
 	(junction
-		(at 167.64 85.09)
-		(diameter 0)
-		(color 0 0 0 0)
-	)
-	(junction
 		(at 104.14 80.01)
 		(diameter 0)
@@
 	(wire
 		(pts
-			(xy 76.2 124.46) (xy 80.01 124.46)
+			(xy 76.2 124.46) (xy 91.44 124.46)
 		)
 		(stroke
@@
 	(wire
 		(pts
+			(xy 167.64 74.93) (xy 167.64 80.01)
+		)
+		(stroke
+			(width 0)
+			(type default)
+		)
+	)
+	(wire
+		(pts
 			(xy 80.01 82.55) (xy 85.09 82.55)
 		)
@@
 		(pts
 			(xy 151.13 97.79) (xy 151.13 99.06)
-		)
-		(stroke
-			(width 0)
-			(type default)
-		)
-	)
-	(wire
-		(pts
-			(xy 91.44 124.46) (xy 87.63 124.46)
 		)
 		(stroke
@@
 	(symbol
 		(lib_id "power:VCC")
-		(at 167.64 85.09 0)
+		(at 167.64 74.93 0)
 		(unit 1)
 		(body_style 1)
@@
 		(dnp no)
 		(property "Reference" "#PWR029"
-			(at 167.64 88.9 0)
+			(at 167.64 78.74 0)
 			(hide yes)
 			(show_name no)
@@
 		)
 		(property "Value" "VCC"
-			(at 168.0718 80.6958 0)
+			(at 168.0718 70.5358 0)
 			(show_name no)
 			(do_not_autoplace no)
@@
 		)
 		(property "Footprint" ""
-			(at 167.64 85.09 0)
+			(at 167.64 74.93 0)
 			(hide yes)
 			(show_name no)
@@
 		)
 		(property "Datasheet" ""
-			(at 167.64 85.09 0)
+			(at 167.64 74.93 0)
 			(hide yes)
 			(show_name no)
@@
 		)
 		(property "Description" ""
-			(at 167.64 85.09 0)
+			(at 167.64 74.93 0)
 			(show_name no)
 			(do_not_autoplace no)
@@
 	)
 	(symbol
+		(lib_id "Device:Fuse_Small")
+		(at 167.64 82.55 270)
+		(unit 1)
+		(body_style 1)
+		(exclude_from_sim no)
+		(in_bom yes)
+		(on_board yes)
+		(in_pos_files yes)
+		(dnp no)
+		(fields_autoplaced yes)
+		(property "Reference" "F1"
+			(at 168.91 81.2799 90)
+			(show_name no)
+			(do_not_autoplace no)
+			(effects
+				(font
+					(size 1.27 1.27)
+				)
+				(justify left)
+			)
+		)
+		(property "Value" "Fuse_Small"
+			(at 168.91 83.8199 90)
+			(show_name no)
+			(do_not_autoplace no)
+			(effects
+				(font
+					(size 1.27 1.27)
+				)
+				(justify left)
+			)
+		)
+		(property "Footprint" "Fuse:Fuse_2512_6332Metric_Pad1.52x3.35mm_HandSolder"
+			(at 167.64 82.55 0)
+			(hide yes)
+			(show_name no)
+			(do_not_autoplace no)
+			(effects
+				(font
+					(size 1.27 1.27)
+				)
+			)
+		)
+		(property "Datasheet" "https://www.littelfuse.com/assetdocs/littelfuse-current-shunt-resistor-ssa-datasheet?assetguid=70d56cd7-0fc3-4a62-93c9-7bee8cc82f45"
+			(at 167.64 82.55 0)
+			(hide yes)
+			(show_name no)
+			(do_not_autoplace no)
+			(effects
+				(font
+					(size 1.27 1.27)
+				)
+			)
+		)
+		(property "Description" "SSA2512L0M20FPR"
+			(at 167.64 82.55 0)
+			(hide yes)
+			(show_name no)
+			(do_not_autoplace no)
+			(effects
+				(font
+					(size 1.27 1.27)
+				)
+			)
+		)
+		(pin "1"
+		)
+		(pin "2"
+		)
+		(instances
+			(project "ads1299_test_board"
+				(path "/97f9a33a-d3bd-406a-9672-b92babffe6b5/a537b4c0-2d82-4fbb-91d8-e3a7ef64a59b"
+					(reference "F1")
+					(unit 1)
+				)
+			)
+		)
+	)
+	(symbol
 		(lib_id "power:GND")
 		(at 167.64 99.06 0)
@@
 	(symbol
 		(lib_id "Switch:SW_Wuerth_450301014042")
-		(at 82.55 88.9 90)
+		(at 82.55 88.9 270)
+		(mirror x)
 		(unit 1)
 		(body_style 1)
@@
 		(dnp no)
 		(property "Reference" "SW1"
-			(at 87.122 90.17 90)
+			(at 77.978 90.17 90)
 			(show_name no)
 			(do_not_autoplace no)
@@
 		)
 		(property "Value" "EG1218"
-			(at 87.63 90.1699 90)
+			(at 77.47 90.1699 90)
 			(hide yes)
 			(show_name no)
@@
 		)
 		(property "Footprint" "Button_Switch_THT:SW_Slide-03_Wuerth-WS-SLTV_10x2.5x6.4_P2.54mm"
-			(at 92.71 88.9 0)
+			(at 72.39 88.9 0)
 			(hide yes)
 			(show_name no)
@@
 		)
 		(property "Datasheet" "https://configured-product-images.s3.amazonaws.com/Datasheets/EG.pdf"
-			(at 90.17 88.9 0)
-			(hide yes)
-			(show_name no)
+			(at 74.93 88.9 0)
+			(hide yes)
+			(show_name no)

Commit message: final
Parts:
- added TP2, TP3, TP3.3v1, TP4, TP5v1: TestPoint, TestPoint:TestPoint_Pad_D1.0mm, symbol Connector:TestPoint
Connections:
- net +3.3V: now also TP3.3v1.1
- net +5V: now also TP5v1.1
- net GND: now also TP2.1, TP3.1
- net VCC: now also TP4.1
