File: ads1299_test_board/ESP32_S3_WROOM.kicad_sch (KiCad schematic)
At the start: 10 parts, among them SW2 SW_MEC_5G, U3 ESP32-S3-WROOM-1

Commit message: GPIO, SRB
Connections:
- net CS: now reaches U3.12 (IO8)
- net GPIO2: now reaches U3.16 (IO46)
- net DOUT: now reaches U3.17 (IO9)
- net DIN: now reaches U3.18 (IO10)
- net SCLK: now reaches U3.19 (IO11)
- net GPIO3: now reaches U3.24 (IO47)
- net GPIO4: now reaches U3.25 (IO48)
- net GPIO1: now reaches U3.26 (IO45)
- net Reset_ads1299: now reaches U3.4 (IO4)
- net Power_ads1299: now reaches U3.5 (IO5)
- net Start: now reaches U3.6 (IO6)
- net DRDY: now reaches U3.7 (IO7)
Other:
- moved on the sheet: C21, C22, C23, C24, SW2

Commit message: updates
Parts:
- C21: footprint (none) -> Capacitor_SMD:C_0603_1608Metric_Pad1.08x0.95mm_HandSolder
- C22, C24: footprint (none) -> Capacitor_SMD:C_0402_1005Metric_Pad0.74x0.62mm_HandSolder
- R20, R21: footprint (none) -> Resistor_SMD:R_0402_1005Metric_Pad0.72x0.64mm_HandSolder
Other:
- moved on the sheet: C24, SW2
Changed lines of the file:
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@@
 	(text "RESET BUTTON "
 		(exclude_from_sim no)
-		(at 27.178 167.132 0)
+		(at 66.548 122.682 0)
 		(effects
 			(font
@@
 	)
 	(junction
-		(at 31.75 180.34)
+		(at 71.12 135.89)
 		(diameter 0)
 		(color 0 0 0 0)
 	)
 	(junction
-		(at 19.05 185.42)
+		(at 58.42 140.97)
 		(diameter 0)
 		(color 0 0 0 0)
@@
 	(polyline
 		(pts
-			(xy 15.24 195.58) (xy 38.1 195.58)
+			(xy 54.61 151.13) (xy 77.47 151.13)
 		)
 		(stroke
@@
 	(wire
 		(pts
-			(xy 19.05 180.34) (xy 21.59 180.34)
-		)
-		(stroke
-			(width 0)
-			(type default)
-		)
-	)
-	(wire
-		(pts
-			(xy 31.75 180.34) (xy 34.29 180.34)
+			(xy 58.42 135.89) (xy 60.96 135.89)
+		)
+		(stroke
+			(width 0)
+			(type default)
+		)
+	)
+	(wire
+		(pts
+			(xy 71.12 135.89) (xy 73.66 135.89)
 		)
 		(stroke
@@
 	(polyline
 		(pts
-			(xy 38.1 195.58) (xy 38.1 170.18)
+			(xy 77.47 151.13) (xy 77.47 125.73)
 		)
 		(stroke
@@
 	(wire
 		(pts
-			(xy 31.75 185.42) (xy 31.75 180.34)
+			(xy 71.12 140.97) (xy 71.12 135.89)
 		)
 		(stroke
@@
 	(wire
 		(pts
-			(xy 30.48 185.42) (xy 31.75 185.42)
+			(xy 69.85 140.97) (xy 71.12 140.97)
 		)
 		(stroke
@@
 	(wire
 		(pts
-			(xy 19.05 185.42) (xy 19.05 187.96)
+			(xy 58.42 140.97) (xy 58.42 143.51)
 		)
 		(stroke
@@
 	(polyline
 		(pts
-			(xy 15.24 170.18) (xy 38.1 170.18)
-		)
-		(stroke
-			(width 0)
-			(type default)
-		)
-	)
-	(wire
-		(pts
-			(xy 19.05 185.42) (xy 22.86 185.42)
+			(xy 54.61 125.73) (xy 77.47 125.73)
+		)
+		(stroke
+			(width 0)
+			(type default)
+		)
+	)
+	(wire
+		(pts
+			(xy 58.42 140.97) (xy 62.23 140.97)
 		)
 		(stroke
@@
 	(wire
 		(pts
-			(xy 19.05 185.42) (xy 19.05 180.34)
+			(xy 58.42 140.97) (xy 58.42 135.89)
 		)
 		(stroke
@@
 	(polyline
 		(pts
-			(xy 15.24 170.18) (xy 15.24 195.58)
+			(xy 54.61 125.73) (xy 54.61 151.13)
 		)
 		(stroke
@@
 	)
 	(label "en"
-		(at 34.29 180.34 0)
+		(at 73.66 135.89 0)
 		(effects
 			(font
@@
 			)
 		)
-		(property "Footprint" ""
+		(property "Footprint" "Capacitor_SMD:C_0603_1608Metric_Pad1.08x0.95mm_HandSolder"
 			(at 108.9152 57.15 0)
 			(hide yes)
@@
 	(symbol
 		(lib_id "power:GNDD")
-		(at 19.05 187.96 0)
+		(at 58.42 143.51 0)
 		(unit 1)
 		(body_style 1)
@@
 		(fields_autoplaced yes)
 		(property "Reference" "#PWR07"
-			(at 19.05 194.31 0)
+			(at 58.42 149.86 0)
 			(hide yes)
 			(show_name no)
@@
 		)
 		(property "Value" "GNDD"
-			(at 19.05 191.77 0)
+			(at 58.42 147.32 0)
 			(show_name no)
 			(do_not_autoplace no)
@@
 		)
 		(property "Footprint" ""
-			(at 19.05 187.96 0)
+			(at 58.42 143.51 0)
 			(hide yes)
 			(show_name no)
@@
 		)
 		(property "Datasheet" ""
-			(at 19.05 187.96 0)
+			(at 58.42 143.51 0)
 			(hide yes)
 			(show_name no)
@@
 		)
 		(property "Description" "Power symbol creates a global label with name \"GNDD\" , digital ground"
-			(at 19.05 187.96 0)
+			(at 58.42 143.51 0)
 			(hide yes)
 			(show_name no)
@@
 			)
 		)
-		(property "Footprint" ""
+		(property "Footprint" "Capacitor_SMD:C_0402_1005Metric_Pad0.74x0.62mm_HandSolder"
 			(at 96.2152 57.15 0)
 			(hide yes)
@@
 			)
 		)
-		(property "Footprint" ""
+		(property "Footprint" "Resistor_SMD:R_0402_1005Metric_Pad0.72x0.64mm_HandSolder"
 			(at 134.62 80.518 90)
 			(hide yes)
@@
 			)
 		)
-		(property "Footprint" ""
+		(property "Footprint" "Resistor_SMD:R_0402_1005Metric_Pad0.72x0.64mm_HandSolder"
 			(at 134.62 75.438 90)
 			(hide yes)
@@
 	(symbol
 		(lib_id "Device:C")
-		(at 26.67 185.42 270)
+		(at 66.04 140.97 270)
 		(unit 1)
 		(body_style 1)
@@
 		(dnp no)
 		(property "Reference" "C24"
-			(at 26.67 189.992 90)
+			(at 66.04 145.542 90)
 			(show_name no)
 			(do_not_autoplace no)
@@
 		)
 		(property "Value" "0.1uF"
-			(at 26.67 192.278 90)
-			(show_name no)
-			(do_not_autoplace no)
-			(effects
-				(font
-					(size 1.27 1.27)
-				)
-			)
-		)
-		(property "Footprint" ""
-			(at 22.86 186.3852 0)
+			(at 66.04 147.828 90)
+			(show_name no)
+			(do_not_autoplace no)
+			(effects
+				(font
+					(size 1.27 1.27)
+				)
+			)
+		)
+		(property "Footprint" "Capacitor_SMD:C_0402_1005Metric_Pad0.74x0.62mm_HandSolder"
+			(at 62.23 141.9352 0)
 			(hide yes)
 			(show_name no)
@@
 		)
 		(property "Datasheet" ""
-			(at 26.67 185.42 0)
+			(at 66.04 140.97 0)
 			(hide yes)
 			(show_name no)
@@
 		)
 		(property "Description" "Unpolarized capacitor"
-			(at 26.67 185.42 0)
+			(at 66.04 140.97 0)
 			(hide yes)
 			(show_name no)
@@
 	(symbol
 		(lib_id "Switch:SW_MEC_5G")
-		(at 26.67 180.34 0)
+		(at 66.04 135.89 0)
 		(unit 1)
 		(body_style 1)
@@
 		(fields_autoplaced yes)
 		(property "Reference" "SW2"
-			(at 26.67 172.72 0)
+			(at 66.04 128.27 0)
 			(show_name no)
 			(do_not_autoplace no)
@@
 		)
 		(property "Value" "SW_MEC_5G"
-			(at 26.67 175.26 0)
+			(at 66.04 130.81 0)
 			(show_name no)
 			(do_not_autoplace no)
@@
 		)
 		(property "Footprint" ""
-			(at 26.67 175.26 0)
+			(at 66.04 130.81 0)
 			(hide yes)
 			(show_name no)
@@
 		)
 		(property "Datasheet" "https://www.apem.com/medias/download/MEC_switches_serie_MULTIMEC5G.pdf"
-			(at 26.67 175.26 0)
+			(at 66.04 130.81 0)
 			(hide yes)
 			(show_name no)
@@
 		)
 		(property "Description" "MEC 5G single pole normally-open tactile switch"
-			(at 26.67 180.34 0)
-			(hide yes)
-			(show_name no)
+			(at 66.04 135.89 0)
+			(hide yes)
+			(show_name no)
