File: ads1299_test_board/ESP32_S3_WROOM.kicad_sch (KiCad schematic)
At the start: 10 parts, among them SW2 SW_MEC_5G, U3 ESP32-S3-WROOM-1

Commit message: PCB design charger and power supply
Connections:
- net CS: now also U3.18 (IO10); no longer U3.12 (IO8)
- net DIN: now also U3.19 (IO11); no longer U3.18 (IO10)
- net DOUT: now also U3.21 (IO13); no longer U3.17 (IO9)
- net DRDY: now also U3.4 (IO4); no longer U3.7 (IO7)
- net Power_ads1299: now also U3.7 (IO7); no longer U3.5 (IO5)
- net Reset_ads1299: now also U3.5 (IO5); no longer U3.4 (IO4)
- net SCLK: now also U3.20 (IO12); no longer U3.19 (IO11)
- net GPIO1: no longer names the net of U3.26 (IO45)
- net GPIO2: no longer names the net of U3.16 (IO46)
- net GPIO3: no longer names the net of U3.24 (IO47)
- net GPIO4: no longer names the net of U3.25 (IO48)
- no-connect marks 8 -> 25

Commit message: final form
Parts:
- removed C14, C20, C23: C, symbol Device:C
Connections:
- net 3.3V: now also C24.1
- net en: no longer C24.1

Commit message: fuse and 1ohm r
Parts:
- removed SW2: SW_MEC_5G, symbol Switch:SW_MEC_5G
- added SW2: PTS810SJM250SMTR LFS, Button_Switch_SMD:SW_SPST_PTS810, symbol Switch:SW_Omron_B3FS
Connections:
- net GNDD: now also SW2.1
- net en: now also SW2.2
Changed lines of the file:
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@@
 	)
 	(symbol
-		(lib_id "Switch:SW_MEC_5G")
+		(lib_id "Switch:SW_Omron_B3FS")
 		(at 66.04 135.89 0)
 		(unit 1)
@@
 			)
 		)
-		(property "Value" "SW_MEC_5G"
+		(property "Value" "PTS810SJM250SMTR LFS"
 			(at 66.04 130.81 0)
 			(show_name no)
@@
 			)
 		)
-		(property "Footprint" ""
+		(property "Footprint" "Button_Switch_SMD:SW_SPST_PTS810"
 			(at 66.04 130.81 0)
 			(hide yes)
@@
 			)
 		)
-		(property "Datasheet" "https://www.apem.com/medias/download/MEC_switches_serie_MULTIMEC5G.pdf"
+		(property "Datasheet" "https://www.littelfuse.com/assetdocs/littelfuse-c-k-tactile-pts810-series-datasheet?assetguid=f1e4bc97-66e9-4beb-99c6-eaef0bd3bff4"
 			(at 66.04 130.81 0)
 			(hide yes)
@@
 			)
 		)
-		(property "Description" "MEC 5G single pole normally-open tactile switch"
+		(property "Description" "Tactile Switch SPST-NO Top Actuated Surface Mount"
 			(at 66.04 135.89 0)
 			(hide yes)
@@
 				)
 			)
-		)
-		(pin "4"
-		)
-		(pin "3"
 		)
 		(pin "1"
@@
 			"5e5913bd-260c-455c-817a-3bac4bc228e8" "5f2e0aed-b4aa-463e-9a5e-0c3fae0711f5"
 			"6366c0cc-1d9d-461e-8903-0ef284a072b5" "9264a05e-565f-4cfd-9732-60272b251642"
-			"d1932d0b-bad0-4ee2-9acb-28daac83eb39" "e2ead138-3d60-48ad-835a-8521441d3c89"
-			"ef12b1bc-83cc-4a22-a750-8b84466cce1c" "fca05337-07ab-4dcf-8821-bcd08aa0a9d1"
+			"d1932d0b-bad0-4ee2-9acb-28daac83eb39" "ef12b1bc-83cc-4a22-a750-8b84466cce1c"
+			"fca05337-07ab-4dcf-8821-bcd08aa0a9d1"
 		)
 	)
