File: ads1299_test_board/ads1299_test_board.kicad_pcb (KiCad board)
At the start: 2 copper layers, 7 parts, among them Q1 AO3407A, U1 ADS1299, U2 MCP73832-2-OT, U3 ESP32-S3-WROOM-1, U4 OPA376xxD, U6 AP2112K-3.3, U7 TPD4E05U06DQA

Commit message: updates
Parts:
- added C1: 10uF, Capacitor_SMD:C_0402_1005Metric_Pad0.74x0.62mm_HandSolder, F.Cu at (148.1, 169.1)
- added C10: 1uF, Capacitor_SMD:C_0402_1005Metric_Pad0.74x0.62mm_HandSolder, F.Cu at (116.0, 155.4)
- added C11: 0.1uF, Capacitor_SMD:C_0402_1005Metric_Pad0.74x0.62mm_HandSolder, F.Cu at (148.1, 173.1)
- added C12: 4.7uF, Capacitor_SMD:C_0402_1005Metric_Pad0.74x0.62mm_HandSolder, F.Cu at (161.6, 155.2)
- added C13: 4.7uF, Capacitor_SMD:C_0402_1005Metric_Pad0.74x0.62mm_HandSolder, F.Cu at (161.6, 157.2)
- added C15: 200pF, Capacitor_SMD:C_0402_1005Metric_Pad0.74x0.62mm_HandSolder, F.Cu at (156.2, 160.0)
- added C16: 10uF, Capacitor_SMD:C_0402_1005Metric_Pad0.74x0.62mm_HandSolder, F.Cu at (156.2, 162.0)
- added C17: 20uF, Capacitor_SMD:C_0805_2012Metric_Pad1.18x1.45mm_HandSolder, F.Cu at (148.9, 155.8)
- added C18: 20uF, Capacitor_SMD:C_0805_2012Metric_Pad1.18x1.45mm_HandSolder, F.Cu at (148.9, 158.8)
- added C19: 20uF, Capacitor_SMD:C_0805_2012Metric_Pad1.18x1.45mm_HandSolder, F.Cu at (148.9, 161.8)
- added C2: 0.15uF, Capacitor_SMD:C_0603_1608Metric_Pad1.08x0.95mm_HandSolder, F.Cu at (112.2, 151.8)
- added C21: 22uF, Capacitor_SMD:C_0603_1608Metric_Pad1.08x0.95mm_HandSolder, F.Cu at (159.9, 169.4)
- added C22: 0.1uF, Capacitor_SMD:C_0402_1005Metric_Pad0.74x0.62mm_HandSolder, F.Cu at (159.4, 171.6)
- added C24: 0.1uF, Capacitor_SMD:C_0402_1005Metric_Pad0.74x0.62mm_HandSolder, F.Cu at (159.4, 173.6)
- added C28: 1uF, Capacitor_SMD:C_0402_1005Metric_Pad0.74x0.62mm_HandSolder, F.Cu at (116.0, 157.4)
- added C3: 0.15uF, Capacitor_SMD:C_0603_1608Metric_Pad1.08x0.95mm_HandSolder, F.Cu at (112.2, 154.3)
- added C4: 0.15uF, Capacitor_SMD:C_0603_1608Metric_Pad1.08x0.95mm_HandSolder, F.Cu at (112.2, 156.8)
- added C5: 0.15uF, Capacitor_SMD:C_0603_1608Metric_Pad1.08x0.95mm_HandSolder, F.Cu at (112.2, 159.3)
- added C6: 100uF, Capacitor_SMD:C_1206_3216Metric_Pad1.33x1.80mm_HandSolder, F.Cu at (152.7, 169.8)
- added C7: 1uF, Capacitor_SMD:C_0402_1005Metric_Pad0.74x0.62mm_HandSolder, F.Cu at (116.0, 151.5)
- added C8: 0.1uF, Capacitor_SMD:C_0402_1005Metric_Pad0.74x0.62mm_HandSolder, F.Cu at (148.1, 171.1)
- added C9: 1uF, Capacitor_SMD:C_0402_1005Metric_Pad0.74x0.62mm_HandSolder, F.Cu at (116.0, 153.5)
- added D1: LED, LED_SMD:LED_0603_1608Metric, F.Cu at (105.5, 167.9)
- added D2: 1N4448W, Diode_SMD:D_SOD-123, F.Cu at (76.2, 121.9)
- added IC1: TPS61023DRLR, Package_TO_SOT_SMD:SOT-563, F.Cu at (156.3, 164.7)
- added IC2: TPS7A2050PDBVR, Package_TO_SOT_SMD:SOT-23-5_HandSoldering, F.Cu at (154.2, 156.7)
- added J1: Conn_01x02, Connector_JST:JST_EH_B2B-EH-A_1x02_P2.50mm_Vertical, F.Cu at (52.0, 158.9)
- added L2: 2.2uH, Inductor_SMD:L_Wuerth_HCI-5040, F.Cu at (60.5, 162.7)
- added P1: USB_C_Plug_USB2.0, Connector_USB:USB_C_Receptacle_G-Switch_GT-USB-7010ASV, F.Cu at (81.0, 171.0)
- added R1: 10K, Resistor_SMD:R_0402_1005Metric_Pad0.72x0.64mm_HandSolder, F.Cu at (105.1, 151.5)
- added R10: 5k, Capacitor_SMD:C_0402_1005Metric_Pad0.74x0.62mm_HandSolder, F.Cu at (161.6, 161.1)
- added R11: 5k, Capacitor_SMD:C_0402_1005Metric_Pad0.74x0.62mm_HandSolder, F.Cu at (161.6, 163.1)
- added R12: 10k, Resistor_SMD:R_0402_1005Metric_Pad0.72x0.64mm_HandSolder, F.Cu at (108.4, 155.5)
- added R14: 100k, Resistor_SMD:R_0402_1005Metric_Pad0.72x0.64mm_HandSolder, F.Cu at (152.9, 160.0)
- added R15: 10k, Resistor_SMD:R_0402_1005Metric_Pad0.72x0.64mm_HandSolder, F.Cu at (83.5, 144.3)
- added R16: 825k, Resistor_SMD:R_0402_1005Metric_Pad0.72x0.64mm_HandSolder, F.Cu at (152.9, 162.0)
- added R17: 10K, Resistor_SMD:R_0402_1005Metric_Pad0.72x0.64mm_HandSolder, F.Cu at (83.5, 146.2)
- added R18: 10k, Resistor_SMD:R_0402_1005Metric_Pad0.72x0.64mm_HandSolder, F.Cu at (83.5, 148.2)
- added R19: 10k, Resistor_SMD:R_0402_1005Metric_Pad0.72x0.64mm_HandSolder, F.Cu at (108.4, 157.5)
- added R2: 10K, Resistor_SMD:R_0402_1005Metric_Pad0.72x0.64mm_HandSolder, F.Cu at (105.1, 153.5)
- added R20: 10K, Resistor_SMD:R_0402_1005Metric_Pad0.72x0.64mm_HandSolder, F.Cu at (111.1, 167.6)
- added R21: 10K, Resistor_SMD:R_0402_1005Metric_Pad0.72x0.64mm_HandSolder, F.Cu at (111.1, 169.6)
- added R22: 5K, Capacitor_SMD:C_0402_1005Metric_Pad0.74x0.62mm_HandSolder, F.Cu at (148.1, 175.0)
- added R24: 5.1K, Capacitor_SMD:C_0402_1005Metric_Pad0.74x0.62mm_HandSolder, F.Cu at (79.2, 163.2)
- added R26: 10k, Resistor_SMD:R_0402_1005Metric_Pad0.72x0.64mm_HandSolder, F.Cu at (108.4, 159.5)
- added R3: 10K, Resistor_SMD:R_0402_1005Metric_Pad0.72x0.64mm_HandSolder, F.Cu at (105.1, 155.5)
- added R4: 10K, Resistor_SMD:R_0402_1005Metric_Pad0.72x0.64mm_HandSolder, F.Cu at (105.1, 157.5)
- added R5: 10K, Resistor_SMD:R_0402_1005Metric_Pad0.72x0.64mm_HandSolder, F.Cu at (105.1, 159.5)
- added R6: 10K, Resistor_SMD:R_0402_1005Metric_Pad0.72x0.64mm_HandSolder, F.Cu at (105.1, 161.4)
- added R7: 10K, Resistor_SMD:R_0402_1005Metric_Pad0.72x0.64mm_HandSolder, F.Cu at (108.4, 151.5)
- added R8: 10K, Resistor_SMD:R_0402_1005Metric_Pad0.72x0.64mm_HandSolder, F.Cu at (108.4, 153.5)
- added R9: 330, Capacitor_SMD:C_0402_1005Metric_Pad0.74x0.62mm_HandSolder, F.Cu at (161.6, 159.2)
- added SW3: SW_SPDT, Button_Switch_THT:SW_Slide_SPDT_Straight_CK_OS102011MS2Q, F.Cu at (93.2, 153.7)
- added TP1: TestPoint, TestPoint:TestPoint_Pad_D1.5mm, F.Cu at (112.0, 162.6)
- moved U7 52.5 mm to (81.8, 163.1), turned to 90 degrees
- moved U1 4.98 mm to (49.8, 96.0), turned to 180 degrees
Connections:
- net Net-(U7-D2+) renamed /USB/Vbus
- U2 pad 4: Vbat -> /USB/Vusb_charge
Routing:
- net GND: track 0.00 -> 0.77 mm
- net /USB/Vbus: track 0.00 -> 0.77 mm
- net /ESP32_S3_WROOM/USB_D-: track 0.00 -> 0.77 mm
- net /ESP32_S3_WROOM/USB_D+: track 0.00 -> 0.77 mm
