File: ads1299_test_board/ads1299_test_board.kicad_pcb (KiCad board)
At the start: 2 copper layers, 67.9 x 57.6 mm, 67 parts, among them CN1 W2A45C103MAT2A, CN2 W2A45C103MAT2A, CN3 W2A45C103MAT2A, CN4 W2A45C103MAT2A, IC1 TPS61023DRLR, IC2 TPS7A2050PDBVR, J1 Conn_01x02, J2 Conn_02x10_Counter_Clockwise, P1 USB_C_Plug_USB2.0, Q1 AO3407A, SW1 EG1218, SW2 PTS810SJM250SMTR LFS, U1 ADS1299, U2 MCP73832-2-OT, U3 ESP32-S3-WROOM-1, U4 OPA376xxD, U6 AP2112K-3.3, U7 TPD4E05U06DQA

Commit message: PCB
Routing:
- net GND: track 43.7 -> 42.4 mm, vias 84 -> 86
- net /ads1299_AFE_/IN1P: track 11.9 -> 11.3 mm
- net /ads1299_AFE_/IN1N: track 14.9 -> 14.4 mm
- removed copper zone on F.Cu, net (none)
Other:
- board size 67.9 x 57.6 mm -> 63.5 x 57.6 mm

Commit message: op-amp sot23-5
Parts:
- removed U4: OPA376xxD, Package_SO:SOIC-8_3.9x4.9mm_P1.27mm
- added U5: OPA376xxDBV, Package_TO_SOT_SMD:SOT-23-5, F.Cu at (131.3, 95.1)
- R10, R11, R9: footprint Capacitor_SMD:C_0402_1005Metric_Pad0.74x0.62mm_HandSolder -> Resistor_SMD:R_0402_1005Metric_Pad0.72x0.64mm_HandSolder
- moved C28 2.43 mm to (133.0, 91.7)
Routing:
- net /ads1299_AFE_/SRB1: track 18.1 -> 15.9 mm
- net /ads1299_AFE_/Ref_electrode: track 31.4 -> 33.3 mm
- net GND: track 42.4 -> 41.1 mm

Commit message: final
Parts:
- added TP2: TestPoint, TestPoint:TestPoint_Pad_D1.0mm, F.Cu at (153.1, 104.0)
- added TP3: TestPoint, TestPoint:TestPoint_Pad_D1.0mm, F.Cu at (169.6, 78.0)
- added TP3.3v1: TestPoint, TestPoint:TestPoint_Pad_D1.0mm, F.Cu at (153.4, 95.6)
- added TP4: TestPoint, TestPoint:TestPoint_Pad_D1.0mm, F.Cu at (164.1, 74.1)
- added TP5v1: TestPoint, TestPoint:TestPoint_Pad_D1.0mm, F.Cu at (156.3, 72.8)
- moved C28 5.79 mm to (138.8, 92.1), turned to -90 degrees
- moved J1 1.38 mm to (170.5, 82.7)
- moved P1 0.82 mm to (169.2, 123.0)
- moved R24 0.82 mm to (163.0, 125.0)
- moved U7 0.82 mm to (162.4, 122.2)
- moved R26 0.61 mm to (146.4, 73.6)
Routing:
- net /ads1299_AFE_/AVDD: track 100.2 -> 87.5 mm
- net GND: track 41.1 -> 52.9 mm, vias 86 -> 85
- net VCC: track 16.2 -> 21.7 mm
- net /ads1299_AFE_/SRB1: track 15.9 -> 17.3 mm
- net /ESP32_S3_WROOM/DOUT: track 26.9 -> 26.3 mm
- net Net-(J1-Pin_2): track 24.1 -> 23.5 mm
- net /ads1299_AFE_/DVDD: track 103.6 -> 104.1 mm, vias 4 -> 2
- added copper zone on F.Cu, net /ads1299_AFE_/AVDD
Other:
- board size 63.5 x 57.6 mm -> 63.5 x 58.4 mm
- board text added: "Big.Brain v 1.0 Rev A"
- board text added: "good luck"
